Commit message: added new robotino modell

File: squirrel_8dof_planner/config/robotino_plan_old.urdf (robot description, URDF)
Before this commit: robot robot, 39 links, 38 joints
Links:
- removed link door_link
- removed link shell_base_link_front
- removed link wheel0_link
- removed link wheel1_link
- removed link wheel2_link
Joints:
- removed joint door_joint
- removed joint shell_base_joint_front
- removed joint wheel0_joint
- removed joint wheel1_joint
- removed joint wheel2_joint
- joint arm_joint1: limit lower=-1.2 upper=1.5 effort=90 velocity=0.7 -> lower=-1.2 upper=-0.55 effort=190 velocity=30
- joint arm_joint2: limit lower=-1.7 upper=2.6 effort=90 velocity=0.7 -> lower=-1.7 upper=2.6 effort=190 velocity=30
- joint arm_joint3: limit lower=-1.8 upper=1.8 effort=90 velocity=0.7 -> lower=-1.8 upper=1.8 effort=190 velocity=30
- joint arm_joint4: limit lower=-2.4 upper=2.4 effort=90 velocity=0.7 -> lower=-2.4 upper=2.4 effort=160 velocity=30
- joint arm_joint5: limit lower=-2.9 upper=2.9 effort=90 velocity=0.7 -> lower=-2.9 upper=2.9 effort=160 velocity=30
