Commit message: added goal pose visualization, services for folding and unfolding, updated srdf to include case

File: squirrel_8dof_planner/config/robotino_plan.urdf (robot description, URDF)
Before this commit: robot robotino, 26 links, 25 joints
Links:
- added link base_neck_link, mass 0.00001; collision box size=0.001 0.001 0.001; visual box size=0.001 0.001 0.001
- added link hand_palm_link
- added link head_link, mass 0.01; collision cylinder length=0.25 radius=0.23; visual mesh filename=package://robotino_description/meshes/head.stl
- added link hokuyo_link, mass 0.00001; collision cylinder length=0.07 radius=0.03; visual mesh filename=package://robotino_description/meshes/hokuyo.dae scale=0.01 0.01 0.01
- added link kinect_link, mass 0.00001; collision box size=0.035 0.18 0.02; visual box size=0.035 0.18 0.02
- added link neck_pan_link, mass 0.01; collision cylinder length=0.08 radius=0.2; visual mesh filename=package://robotino_description/meshes/neck.stl
- added link neck_tilt_link, mass 0.01
- added link shell_base_link, mass 0.01; collision mesh filename=package://robotino_description/meshes/base_shell_collision.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; visual mesh filename=package://robotino_description/meshes/base_shell.stl
- link base_link: mass None -> 10
Joints:
- added joint base_neck_joint: type fixed, parent base_link, child base_neck_link, origin xyz=0.0 0.0 0.676 rpy=0.0 0.0 0.0
- added joint hand_palm_joint: type fixed, parent hand_wrist_link, child hand_palm_link, origin xyz=-0.02105 0.2485 0 rpy=-1.5708 0 0
- added joint head_joint: type revolute, parent base_link, child head_link, origin xyz=0 0 0.715 rpy=0 0 0, axis 0 0 -1, limit lower=-3.14 upper=3.14 effort=100 velocity=1.4
- added joint hokuyo_joint: type fixed, parent base_link, child hokuyo_link, origin xyz=0.184 0.004 0.1 rpy=0.0 0.0 -0.015
- added joint kinect_joint: type fixed, parent neck_tilt_link, child kinect_link, origin xyz=0.0 0.0 0.0 rpy=-1.57 0.0 0.0
- added joint neck_pan_joint: type revolute, parent base_neck_link, child neck_pan_link, origin xyz=0 0 0 rpy=0 0 0, axis 0 0 -1, limit lower=-3.14 upper=3.14 effort=100 velocity=1.4
- added joint neck_tilt_joint: type revolute, parent neck_pan_link, child neck_tilt_link, origin xyz=0.192 0 0 rpy=1.57 0 0, axis 0 0 1, limit lower=-1.19 upper=0.52 effort=100 velocity=1.4
- added joint shell_base_joint: type fixed, parent base_link, child shell_base_link, origin xyz=0.0 0.0 0.0 rpy=0.0 0.0 0.0
- joint arm_base_joint: origin xyz=0.0 -0.01591 0.32 rpy=0.0 0.0 -1 -> xyz=0.0 -0.01591 0.25 rpy=0.0 0.0 -1
- joint arm_joint1: axis 0 1 0 -> 0 -1 0; limit lower=-1.9 upper=1.9 effort=190 velocity=30 -> lower=-1.2 upper=1.5 effort=190 velocity=30
- joint arm_joint2: limit lower=-1.9 upper=1.9 effort=190 velocity=30 -> lower=-1.7 upper=2.6 effort=190 velocity=30
- joint arm_joint3: limit lower=-1.7 upper=1.7 effort=190 velocity=30 -> lower=-1.8 upper=1.8 effort=190 velocity=30
- joint arm_joint4: axis 0 1 0 -> 0 -1 0; limit lower=-1.7 upper=1.7 effort=160 velocity=30 -> lower=-2.4 upper=2.4 effort=160 velocity=30
- joint arm_joint5: limit lower=-1.7 upper=1.7 effort=160 velocity=30 -> lower=-2.9 upper=2.9 effort=160 velocity=30

Commit message: removed collision between arm_joint_1 and base_link

File: squirrel_8dof_planner/config/robotino_plan.urdf (robot description, URDF)
Before this commit: robot robotino, 34 links, 33 joints
Joints:
- joint base_theta_joint: origin xyz=0 0 0 rpy=0 0 0 -> xyz=0.00001 0.00001 0.00001 rpy=0 0 0

Commit message: changed folding trajectory be per robot, updated launchfile and disabled collisions with virtual joints

File: squirrel_8dof_planner/config/robotino_plan.urdf (robot description, URDF)
Before this commit: robot robotino, 34 links, 33 joints
Joints:
- joint base_theta_joint: origin xyz=0.00001 0.00001 0.00001 rpy=0 0 0 -> xyz=0 0 0 rpy=0 0 0

Commit message: fixed wrong initializer for goal pose finding

File: squirrel_8dof_planner/config/robotino_plan.urdf (robot description, URDF)
Before this commit: robot robotino, 34 links, 33 joints
Joints:
- joint arm_joint1: limit lower=-1.2 upper=1.5 effort=190 velocity=30 -> lower=-1.2 upper=-0.55 effort=190 velocity=30

Commit message: added collision visualization and corrected internal link collision transforms for collision modell

File: squirrel_8dof_planner/config/robotino_plan.urdf (robot description, URDF)
Before this commit: robot robot, 39 links, 38 joints
Links:
- link wheel0_link: geometry visual mesh filename=package://robotino_description/meshes/RobotinoWheel.dae scale=0.01 0.01 0.01
- link wheel1_link: geometry visual mesh filename=package://robotino_description/meshes/RobotinoWheel.dae scale=0.01 0.01 0.01
- link wheel2_link: geometry visual mesh filename=package://robotino_description/meshes/RobotinoWheel.dae scale=0.01 0.01 0.01

Commit message: minor

File: squirrel_8dof_planner/config/robotino_plan.urdf (robot description, URDF)
Before this commit: robot robot, 39 links, 38 joints
Links:
- link shell_base_link_front: geometry collision box size=0.55 0.55 0.17
